File: Power Supply.kicad_sch (KiCad schematic)
At the start: 80 parts, among them J10 Connector, J11 Connector, J12 Connector, J13 Connector, J14 Connector, J15 Connector, J16 Connector, J17 Connector, J18 Connector, J19 Connector, J20 Connector, J23 Connector, J24 Connector, J25 Connector, J26 Connector, J27 Connector, J28 Connector, J29 Connector, J3 Connector, J30 Connector, J31 Connector, J32 Connector, J33 Connector, J34 Connector, J4 Connector, J5 Connector, J6 Connector, J7 Connector, J8 Connector, J9 Connector, M1 TDK, M2 TDK, M3 TDK

Commit message: Power Supplie Board V1.00
Parts:
- C1, C2, C5: footprint (none) -> Capacitor_SMD:CP_Elec_4x5.8
- C10, C7, C8, C9: footprint (none) -> Capacitor_THT:CP_Radial_D8.0mm_P5.00mm
- C11, C12, C13, C14, C15, C16, C17, C18, C19, C20, C21, C22, C23, C24, C25, C26, C27, C28, C29, C30, C31, C32, C33, C34, C35, C36, C37, C38, C39, C40: footprint (none) -> Capacitor_THT:C_Disc_D7.5mm_W5.0mm_P5.00mm
- C3, C4, C6: footprint (none) -> Capacitor_SMD:CP_Elec_4x5.7
- J1, J2, J21, J22: footprint (none) -> My Global Library:7461383
- J10, J11, J12, J13, J14, J15, J16, J17, J18, J19, J20, J23, J24, J25, J26, J27, J28, J29, J3, J30, J31, J32, J33, J34, J4, J5, J6, J7, J8, J9: footprint (none) -> Connector_JST:JST_EH_B2B-EH-A_1x02_P2.50mm_Vertical
- M1, M2, M3: footprint I3A4W005A150V001R -> My Global Library:I3A4W005A150V001R
- R1, R2, R3: footprint (none) -> Resistor_THT:R_Axial_DIN0204_L3.6mm_D1.6mm_P7.62mm_Horizontal
Connections:
- net +12V: no longer C31.1, C32.1, C33.1, C34.1, C35.1, C36.1, C37.1, C38.1, C39.1, C40.1, C5.1, C6.1, J15.1 (Pin_1), J16.1 (Pin_1), J17.1 (Pin_1), J18.1 (Pin_1), J19.1 (Pin_1), J20.1 (Pin_1), J31.1 (Pin_1), J32.1 (Pin_1), J33.1 (Pin_1), J34.1 (Pin_1), M3.7 (SENSE_(+)), M3.8 (VOUT_(+))
- net +6V: now also M2.8 (V_{OUT}+)
- net GND1: now also M2.4 (V_{OUT}-)
- new net Vdrive: C31.1, C32.1, C33.1, C34.1, C35.1, C36.1, C37.1, C38.1, C39.1, C40.1, C5.1, C6.1, J15.1 (Pin_1), J16.1 (Pin_1), J17.1 (Pin_1), J18.1 (Pin_1), J19.1 (Pin_1), J20.1 (Pin_1), J31.1 (Pin_1), J32.1 (Pin_1), J33.1 (Pin_1), J34.1 (Pin_1), M3.7 (SENSE_(+)), M3.8 (VOUT_(+))
Other:
- moved on the sheet: C1, C4
